Commit message: Delete node_practice directory

File: cobot_simulation/urdf/cobot.urdf (robot description, URDF)
Before this commit: robot cobot, 0 links, 0 joints
Links:
- added link world
Joints:
- added joint fixed: type fixed, parent world, child base_link

File: cobot_simulation/urdf/joint_link.xacro (robot description, xacro)
@@ -52,17 +52,17 @@
         </joint>
     </xacro:macro>
-     <!-- <xacro:macro name="transmission" params="name joint_name actuator_name">
+     <xacro:macro name="transmission" params="name joint_name actuator_name">
         <transmission name="${name}" >
             <type>transmission_interface/SimpleTransmission</type>
             <joint name = "${joint_name}" >
-                <hardwareInterface>hardware_interface/PositionJointInterface</hardwareInterface>
+                <hardwareInterface>hardware_interface/EffortJointInterface</hardwareInterface>
             </joint>
             <actuator name="${actuator_name}" >
-                <hardwareInterface>hardware_interface/PositionJointInterface</hardwareInterface>
+                <hardwareInterface>hardware_interface/EffortJointInterface</hardwareInterface>
                 <mechanicalReduction>1</mechanicalReduction>
             </actuator>
         </transmission>
     </xacro:macro>
-    <xacro:macro name="transmission_effort" params="name joint_name actuator_name">
+    <!-- <xacro:macro name="transmission_effort" params="name joint_name actuator_name">
         <transmission name="${name}" >
             <type>transmission_interface/SimpleTransmission</type>
@@ -76,8 +76,3 @@
         </transmission>
     </xacro:macro> -->
-     <!-- <gazebo>
-        <plugin name="gazebo_ros_control" filename="libgazebo_ros_control.so">
-            <robotNamespace>/cobot</robotNamespace>
-        </plugin>
-    </gazebo> -->
 </robot>
