Commit message: nambah

File: cobot_simulation/urdf/gripper.xacro (robot description, xacro)
@@ -5,5 +5,5 @@
     <xacro:macro name="gripper" params="parent origin_xyz">
         <!-- Gripper connector-->
-        <xacro:cobot_link_box name="gripper_connector" origin_xyz="0.0 0.0 0.0125" origin_rpy="0 0 0"
+        <xacro:cobot_link_box name="gripper_connector" origin_xyz="0.0 0.0 0.035" origin_rpy="0 0 0"
                             size="0.03 0.150 0.03"
                             mass="1" ixx="0.00195" ixy="0" ixz="0" iyy="0.00195" iyz="0" izz="0.00015"/>
@@ -52,4 +52,42 @@
                         joint_name="gripper_left_joint"
                         actuator_name="motor_gripper_left_joint" />
- </xacro:macro>
+        <!-- ros control plugin with mimic-->
+        <xacro:macro name="mimic_joint_plugin_gazebo" params="parent_joint mimic_joint has_pid:=false multiplier:=-1.0 offset:=0 sensitiveness:=0.0 max_effort:=200 robot_namespace:='/cobot'">
+            <gazebo>
+                <plugin name="${mimic_joint}_mimic_joint_plugin" filename="libroboticsgroup_gazebo_mimic_joint_plugin.so">
+                    <joint>${parent_joint}</joint>
+                    <mimicJoint>${mimic_joint}</mimicJoint>
+                    <xacro:if value="${has_pid}">
+                        <hasPID />
+                    </xacro:if>
+                    <multiplier>${multiplier}</multiplier>
+                    <offset>${offset}</offset>
+                    <sensitiveness>${sensitiveness}</sensitiveness>
+                    <maxEffort>${max_effort}</maxEffort>
+                    <xacro:unless value="${robot_namespace == '/cobot'}">
+                        <robotNamespace>($robot_namespace)</robotNamespace>
+                    </xacro:unless>
+                </plugin>
+            </gazebo>
+        </xacro:macro>
+        <xacro:mimic_joint_plugin_gazebo  parent_joint="gripper_right_joint" mimic_joint="gripper_left_joint"
+                                            has_pid="false" multiplier="-1.0" max_effort="200" />
+        <gazebo>
+            <plugin name="gazebo_grasp_fix" filename="libgazebo_grasp_fix.so">
+                <arm>
+                    <arm_name>gripper</arm_name>
+                    <palm_link>gripper_connector</palm_link>
+                    <gripper_link> gripper_right </gripper_link>
+                    <gripper_link> gripper_left </gripper_link>
+                </arm>
+                <forces_angle_tolerance>100</forces_angle_tolerance>
+                <update_rate>10</update_rate>
+                <grip_count_threshold>3</grip_count_threshold>
+                <max_grip_count>10</max_grip_count>
+                <release_tolerance>0.001</release_tolerance>
+                <disable_collision_on_attach>false</disable_collision_on_attach>
+                <contact_topic>__default_topic__</contact_topic>
+            </plugin>
+        </gazebo>
+    </xacro:macro>
 </robot>

File: cobot_simulation/urdf/joint_link.xacro (robot description, xacro)
@@ -56,8 +56,8 @@
             <type>transmission_interface/SimpleTransmission</type>
             <joint name = "${joint_name}" >
-                <hardwareInterface>hardware_interface/EffortJointInterface</hardwareInterface>
+                <hardwareInterface>hardware_interface/PositionJointInterface</hardwareInterface>
             </joint>
             <actuator name="${actuator_name}" >
-                <hardwareInterface>hardware_interface/EffortJointInterface</hardwareInterface>
+                <hardwareInterface>hardware_interface/PositionJointInterface</hardwareInterface>
                 <mechanicalReduction>1</mechanicalReduction>
             </actuator>
